Commit message: w2_sim: 忠实仿真 RoboSense AIRY 雷达(替换 OS1 近似)
把 Isaac 仿真雷达从内置 OS1_REV6_32ch10hz1024res(±22° 垂直 FOV、3.2万点)
改为忠实的 RoboSense AIRY:96 线、垂直 FOV 0~90° 半球穹顶(0.947° 均布)、
水平 360° @ 0.4°(900 方位步)、测距 0.1~60m、距离精度 1.5cm(1σ)、单回波。

雷达 config:
- Isaac Sim 5.x RTX lidar 不再用本地 JSON;config= 只解析资产服务器 USD 名,
  真实参数在 OmniLidar prim 的 omni:sensor:Core:* 属性。
- 实测插件解析 emitter 配置时不读 stage 合成后的属性,而是顺 prim 的 reference/
  payload 读原始资产(OS1→payload 32 线、Example_Rotary→reference 128 线),
  就地覆写/引用/flatten 都无效(报 "NumberOfEmitters 96 != 32/128" 崩溃)。
- 解决:isaac/make_airy_usd.py 用 Example_Rotary 模板就地覆写成 96 线 AIRY 后
  flatten 导出 config/RS_Airy.usd(concrete spec、无 reference/payload);主程序
  用 Sdf.CopySpec 把该 prim spec 物理拷进 stage,插件读到完整 96 线 AIRY 配置。
- 必须重置全部 11 个 per-emitter 数组到长度 96(不止 elevation;focalDistM/
  focalSlope/horOffsetM/vertOffsetM/reportRateDiv 默认 128,漏改即崩)。

安装外参(真机竖直安装,改自占位错值 58° 前倾):
- 读 finder_lidar_mapping/glim_ros2/launch/airy_tf_tree.launch.py,复合
  base_link→imu_link RPY 与 imu_link→rslidar 四元数,得 base_link→rslidar 旋转
  ≈ 单位阵(rslidar +Z ≈ base +Z 朝上,半球穹顶朝上,符合补盲)。路 (a):改 URDF
  rslidar joint rpy 1.01→0、重导 USD、同步 demo_episode.sh static TF。

验证(无头,对照真实 bag /rslidar_points):
  仿真 el[0,89.96]° az[0,360]° ~84.7k 点 96 层;真实 el[-0.2,88.5]° az 360°
  ~64k 点(场景受限)96×900。el 上半球覆盖、点数量级、层数全吻合。
  rate 仿真 ~2.4Hz(sim-clock,渲染吞吐受限于 86k 射线,非配置错误)vs 真机 9.55Hz。
  intensity/ring/timestamp 暂未加(ROS2RtxLidarHelper point_cloud 仅出 xyz,
  加这些字段需自定义 annotator+writer 链,代价大,本次未做)。

Co-Authored-By: Claude Opus 4.8 (1M context) <noreply@anthropic.com>

File: w2_sim/urdf/W2EVT1Urdf_swerve.urdf.xacro (robot description, xacro)
@@ -70,11 +70,16 @@
   <xacro:swerve_module prefix="rear_left"   x="${-wheelbase/2}" y="${ track_width/2}"/>
   <xacro:swerve_module prefix="rear_right"  x="${-wheelbase/2}" y="${-track_width/2}"/>
-  <!-- 传感器帧。倾角为近似值(design §4:精确外参非本期关键);
-       Task 11 验证步骤会用实车静止段重力方向校核倾角符号。 -->
+  <!-- 传感器帧。
+       rslidar:RoboSense AIRY 竖直安装(半球穹顶 FOV 沿传感器 +Z 朝上)。
+       真机外参取自 finder_lidar_mapping/glim_ros2/launch/airy_tf_tree.launch.py:
+       base_link→imu_link RPY(3.1415,0,-1.5708) 复合 imu_link→rslidar 四元数
+       (0.7098,-0.7044,0.0050,-0.0015) 后,base_link→rslidar 旋转 ≈ 单位阵
+       (残差 <0.01 rad,属标定噪声),即 rslidar +Z ≈ base +Z(朝上)。
+       位置 xyz(0.25,0,0.55) 为合理估计(真机标定平移仅毫米级,可忽略)。 -->
   <link name="rslidar"/>
   <joint name="base_link_to_rslidar" type="fixed">
     <parent link="base_link"/>
     <child  link="rslidar"/>
-    <origin xyz="0.25 0 0.55" rpy="0 1.01 0"/>  <!-- pitch ~58° 前倾(近似) -->
+    <origin xyz="0.25 0 0.55" rpy="0 0 0"/>  <!-- AIRY 竖直安装,半球穹顶朝上 -->
   </joint>
   <link name="imu_link"/>
